File: bifrost.kicad_pcb (KiCad board)
At the start: 2 copper layers, 366.7 x 119.1 mm, 322 parts, among them J1 USB_C_Receptacle, J2 AVR-ISP-6, SW1 SW_SPST, SW10 SW_SPST, SW100 SW_SPST, SW101 SW_SPST, SW11 SW_SPST, SW12 SW_SPST, SW13 SW_SPST, SW14 SW_SPST, SW15 SW_SPST, SW16 SW_SPST, SW17 SW_SPST, SW18 SW_SPST, SW19 SW_SPST, SW2 SW_SPST, SW20 SW_SPST, SW21 SW_SPST, SW22 SW_SPST, SW23 SW_SPST, SW24 SW_SPST, SW25 SW_SPST, SW26 SW_SPST, SW27 SW_SPST, SW28 SW_SPST, SW29 SW_SPST, SW3 SW_SPST, SW30 SW_SPST, SW31 SW_SPST, SW32 SW_SPST, SW33 SW_SPST, SW34 SW_SPST, SW35 SW_SPST, SW36 SW_SPST, SW37 SW_SPST, SW38 SW_SPST, SW39 SW_SPST, SW4 SW_SPST, SW40 SW_SPST, SW41 SW_SPST, SW42 SW_SPST, SW43 SW_SPST, SW44 SW_SPST, SW45 SW_SPST, SW46 SW_SPST, SW47 SW_SPST, SW48 SW_SPST, SW49 SW_SPST, SW5 SW_SPST, SW50 SW_SPST, SW51 SW_SPST, SW52 SW_SPST, SW53 SW_SPST, SW54 SW_SPST, SW55 SW_SPST, SW56 SW_SPST, SW57 SW_SPST, SW58 SW_SPST, SW59 SW_SPST, SW6 SW_SPST, SW60 SW_SPST, SW65 SW_SPST, SW66 SW_SPST, SW67 SW_SPST, SW68 SW_SPST, SW69 SW_SPST, SW7 SW_SPST, SW70 SW_SPST, SW71 SW_SPST, SW72 SW_SPST, SW73 SW_SPST, SW74 SW_SPST, SW75 SW_SPST, SW76 SW_SPST, SW77 SW_SPST, SW78 SW_SPST, SW79 SW_SPST, SW8 SW_SPST, SW80 SW_SPST, SW81 SW_SPST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

Commit message: save before diddelidoo
Parts:
- C1, C2, C3, C4, C5, D100, D101, D102, D103, D104, D105, D106, D107, D108, D109, D110, D111, D112, D113, D114, D115, D116, D117, D118, D119, D120, D121, D122, D123, D124, D177, D178, D179, D180, D181, D182, D183, D184, D185, D186, D187, D188, D189, D190, D191, D192, D193, D194, D195, D196, D197, D198, D199, D200, D201, D202, D203, D204, D205, D206, D207, D208, D209, D210, D211, D212, D213, D65, D66, D67, D68, D69, D70, D71, D72, D73, D74, D75, D76, D77, D78, D79, D80, D81, D82, D83, D84, D85, D86, D87, D88, D89, D90, D91, D92, D93, D94, D95, D96, D97, D98, D99, F1, L1, R1, R2, R3, R4, R5, U1, Y1: moved to B.Cu
- moved J1 384.4 mm to (304.8, -7.14), turned to 180 degrees
- moved D208 373.5 mm to (383.4, 31.0), turned to 90 degrees
- moved D207 358.2 mm to (383.4, 7.14), turned to 90 degrees
- moved D206 356.9 mm to (364.3, 7.14), turned to 90 degrees
- moved D115 349.5 mm to (364.3, 31.0), turned to 90 degrees
- moved R4 349.2 mm to (300.0, 19.1), turned to 270 degrees
- moved R1 344.6 mm to (302.4, 4.16)
- moved L1 342.6 mm to (304.8, 9.53)
- moved D113 337.7 mm to (326.2, 31.0), turned to 90 degrees
- moved D181 333.4 mm to (295.3, 14.3), turned to 90 degrees
- moved D210 329.2 mm to (383.4, 59.5), turned to 90 degrees
- moved D65 317.3 mm to (35.7, 7.14), turned to 90 degrees
- moved D72 313.3 mm to (197.6, 7.14), turned to 90 degrees
- moved C5 310.4 mm to (294.5, 21.4)
- moved D66 310.0 mm to (73.8, 7.14), turned to 90 degrees
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Routing:
- net F: track 0.00 -> 300.0 mm
- net A: track 0.00 -> 266.7 mm
- net B: track 0.00 -> 257.2 mm
- net E: track 0.00 -> 247.7 mm
- net D: track 0.00 -> 235.7 mm
- net C: track 0.00 -> 233.4 mm
- net G: track 0.00 -> 178.9 mm
- net Net-(D158-Pad4): track 0.00 -> 65.4 mm
- net Net-(D157-Pad4): track 0.00 -> 65.4 mm
- net H: track 0.00 -> 63.3 mm
- net Net-(D16-Pad4): track 0.00 -> 32.1 mm
- net Net-(D137-Pad4): track 0.00 -> 29.7 mm
- net Net-(D22-Pad4): track 0.00 -> 22.6 mm
- net Net-(D12-Pad4): track 0.00 -> 22.6 mm
- net Net-(D8-Pad4): track 0.00 -> 22.6 mm
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
Commit message: complete makeover
Parts:
- removed D162, D163, D164, D165, D166, D167, D168, D169, D170, D171, D172, D173, D174, D175, D176: SK6812, misc:SK6812_IN-PCB
- moved D149 326.8 mm to (354.8, 59.5), turned to 180 degrees
- moved D161 305.0 mm to (316.7, -2.38)
- moved D160 300.5 mm to (335.8, -2.38)
- moved D159 296.0 mm to (354.8, -2.38)
- moved D148 286.4 mm to (335.8, 59.5), turned to 180 degrees
- moved D134 279.3 mm to (76.2, 97.6), turned to 180 degrees
- moved D18 271.5 mm to (102.4, 21.4), turned to 180 degrees
- moved D147 248.4 mm to (316.7, 59.5), turned to 180 degrees
- moved D158 247.3 mm to (373.9, -2.38)
- moved D19 233.4 mm to (121.4, 21.4), turned to 180 degrees
- moved D143 228.8 mm to (373.9, 88.1)
- moved D145 228.6 mm to (335.8, 78.6)
- moved D146 228.6 mm to (316.7, 78.6)
- moved D144 228.6 mm to (354.8, 78.6)
- moved D37 223.8 mm to (111.9, 40.5)
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Connections:
- D108 pad 1: 4 -> 7
- D109 pad 1: 5 -> 11
- D110 pad 1: 6 -> 12
- D111 pad 1: 7 -> 13
- D112 pad 1: 8 -> 14
- D113 pad 1: 1 -> 15
- D114 pad 1: 2 -> 16
- D115 pad 1: 3 -> 17
- D116 pad 1: 4 -> 15
- D117 pad 1: 5 -> 16
- D118 pad 1: 6 -> 17
- D119 pad 1: 7 -> 15
- D120 pad 1: 8 -> 16
- D121 pad 1: 1 -> 15
- D122 pad 1: 2 -> 16
- D123 pad 1: 3 -> 17
- D124 pad 1: 4 -> 18
- D182 pad 1: 14 -> 15
- D204 pad 1: 9 -> 14
- D205 pad 1: 10 -> 16
- D206 pad 1: 11 -> 17
- D207 pad 1: 12 -> 18
- D208 pad 1: 13 -> 18
- D209 pad 1: 9 -> 17
- D210 pad 1: 10 -> 18
- D211 pad 1: 11 -> 15
- D212 pad 1: 12 -> 16
- D213 pad 1: 13 -> 17
- SW100 pad 1: G -> E
- SW101 pad 1: G -> E
- SW49 pad 1: G -> B
- SW50 pad 1: G -> B
- SW51 pad 1: G -> B
- SW52 pad 1: G -> C
- SW53 pad 1: G -> C
- SW54 pad 1: G -> C
- SW55 pad 1: G -> D
- SW56 pad 1: G -> D
- SW57 pad 1: H -> F
- SW58 pad 1: H -> F
- SW59 pad 1: H -> F
- SW60 pad 1: H -> E
- SW92 pad 1: F -> C
- SW93 pad 1: F -> A
- SW94 pad 1: F -> A
- SW95 pad 1: F -> A
- SW96 pad 1: F -> B
- SW97 pad 1: G -> D
- SW98 pad 1: G -> C
- SW99 pad 1: G -> E
- U1 pad 15: Net-(U1-Pad15) -> GND
- U1 pad 18: A -> 11
- U1 pad 19: B -> 12
- U1 pad 20: C -> 13
- U1 pad 21: D -> 14
- U1 pad 22: F -> 16
- U1 pad 23: Net-(U1-Pad15) -> GND
- U1 pad 25: E -> 15
- U1 pad 26: G -> 17
- U1 pad 27: H -> 18
- U1 pad 31: Net-(U1-Pad31) -> 9
- U1 pad 32: Net-(U1-Pad32) -> 10
- U1 pad 35: Net-(U1-Pad15) -> GND
- U1 pad 36: 14 -> F
- U1 pad 37: 13 -> E
- U1 pad 38: 12 -> D
- U1 pad 39: 11 -> C
- U1 pad 40: 10 -> B
- U1 pad 41: 9 -> A
- U1 pad 43: Net-(U1-Pad15) -> GND
- U1 pad 5: Net-(U1-Pad5) -> GND
Routing:
- net +5V: track 0.00 -> 1849.5 mm, vias 0 -> 66
- net 1: track 0.00 -> 375.2 mm, vias 0 -> 16
- net 2: track 0.00 -> 370.4 mm, vias 0 -> 19
- net 3: track 0.00 -> 355.9 mm, vias 0 -> 20
- net 4: track 0.00 -> 310.9 mm, vias 0 -> 16
- net 5: track 0.00 -> 291.1 mm, vias 0 -> 16
- net 6: track 0.00 -> 272.6 mm, vias 0 -> 16
- net 7: track 0.00 -> 271.2 mm, vias 0 -> 20
- net 8: track 0.00 -> 230.5 mm, vias 0 -> 16
- net 9: track 0.00 -> 210.4 mm, vias 0 -> 16
- net 11: track 0.00 -> 195.1 mm, vias 0 -> 20
- net 10: track 0.00 -> 192.7 mm, vias 0 -> 16
- net G: track 178.9 -> 0.00 mm
- net 12: track 0.00 -> 175.3 mm, vias 0 -> 20
- net 13: track 0.00 -> 110.6 mm, vias 0 -> 16
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- added copper zone on F.Cu, net GND
Other:
- net class GND added: clearance 0.5, trace_width 0.5, via_dia 0.8, via_drill 0.4

Commit message: rev0
Parts:
- J2: value AVR-ISP-6 -> Conn_02x04_Counter_Clockwise; footprint Connector_PinHeader_2.54mm:PinHeader_2x03_P2.54mm_Vertical -> misc:SOIC_clipProgSmall
- moved J2 88.0 mm to (373.4, 111.5), turned to 0 degrees
- moved R3 20.6 mm to (305.8, 2.03)
- moved R4 20.5 mm to (303.7, 2.03)
- moved C5 17.1 mm to (309.4, 15.2)
- moved Y1 13.6 mm to (301.2, 33.5), turned to 0 degrees
- moved U1 12.7 mm to (300.7, 18.3), turned to 180 degrees
- moved C2 10.5 mm to (299.2, 27.9), turned to 0 degrees
- moved F1 5.88 mm to (301.2, 4.06)
- moved C1 5.75 mm to (311.4, 13.2)
- moved C3 5.55 mm to (303.3, 27.9), turned to 180 degrees
- moved R5 5.00 mm to (307.3, 27.9), turned to 0 degrees
- moved C4 4.07 mm to (309.9, 22.9)
- moved R2 3.75 mm to (307.8, 2.03)
- moved L1 2.13 mm to (302.8, 9.14), turned to 0 degrees
- moved D181 1.02 mm to (295.7, 9.65)
Connections:
- J2 pad 1: 4 -> +5V
- J2 pad 2: +5V -> Net-(J2-Pad2)
- J2 pad 3: 2 -> Net-(J2-Pad3)
- J2 pad 4: 3 -> GND
- J2 pad 5: Net-(J2-Pad5) -> 17
- J2 pad 6: GND -> 18
- R5 pad 2: Net-(J2-Pad5) -> Net-(J2-Pad8)
- U1 pad 10: 3 -> 17
- U1 pad 11: 4 -> 18
- U1 pad 12: 8 -> 14
- U1 pad 13: Net-(J2-Pad5) -> Net-(J2-Pad8)
- U1 pad 18: 11 -> 13
- U1 pad 19: 12 -> 1
- U1 pad 20: 13 -> 2
- U1 pad 21: 14 -> 3
- U1 pad 22: 16 -> 4
- U1 pad 25: 15 -> 5
- U1 pad 26: 17 -> 6
- U1 pad 27: 18 -> 7
- U1 pad 28: 5 -> 8
- U1 pad 29: 6 -> 9
- U1 pad 30: 7 -> 10
- U1 pad 31: 9 -> 11
- U1 pad 32: 10 -> 12
- U1 pad 8: 1 -> 15
- U1 pad 9: 2 -> 16
Routing:
- net +5V: track 1849.5 -> 2511.1 mm, vias 66 -> 116
- net E: track 247.7 -> 456.0 mm, vias 0 -> 8
- net 16: track 0.00 -> 190.1 mm, vias 0 -> 18
- net 18: track 0.00 -> 188.1 mm, vias 0 -> 8
- net 17: track 0.00 -> 187.7 mm, vias 0 -> 16
- net F: track 261.9 -> 438.0 mm, vias 0 -> 8
- net Net-(J2-Pad8): track 0.00 -> 162.2 mm, vias 0 -> 8
- net C: track 263.5 -> 408.9 mm, vias 0 -> 5
- net D: track 235.7 -> 380.3 mm, vias 0 -> 9
- net 15: track 0.00 -> 135.7 mm, vias 0 -> 16
- net B: track 257.2 -> 366.4 mm, vias 0 -> 5
- net A: track 266.7 -> 354.7 mm, vias 0 -> 3
- net 13: track 110.6 -> 163.7 mm, vias 16 -> 18
- net Net-(D27-Pad4): track 0.00 -> 41.4 mm, vias 0 -> 6
- net Net-(D54-Pad4): track 0.00 -> 33.2 mm, vias 0 -> 4
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- added copper zone on B.Cu, net GND
Other:
- board size 366.7 x 119.1 mm -> 366.7 x 123.8 mm
- net class GND: clearance 0.5 -> 0.2
- net class soicbyte added: clearance 0.05, trace_width 0.2, via_dia 0.8, via_drill 0.4
